File: PCBs/keezer_pcb/esp32_smart_keezer.kicad_pcb (KiCad board)
At the start: 2 copper layers, 67.8 x 59.3 mm, 39 parts, among them J1 Conn_01x03_Male, J10 Conn_01x03_Male, J11 USB_B_Micro, J2 Conn_01x03_Male, J3 Conn_01x03_Male, J4 Conn_01x03_Male, J5 Conn_01x03_Male, J6 Conn_01x03_Male, J7 Conn_01x03_Male, J8 Conn_01x03_Male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

Commit message: Rev 1 - WIP
Parts:
- removed R25: 200R, Resistor_SMD:R_0603_1608Metric
- removed R26: 330R, Resistor_SMD:R_0603_1608Metric
- added C4: 0.47uF, Capacitor_SMD:C_0805_2012Metric, F.Cu at (174.3, 105.2)
- added C5: 10u, Capacitor_SMD:C_0805_2012Metric, F.Cu at (167.4, 101.2)
- added C6: 10u, Capacitor_SMD:C_0805_2012Metric, F.Cu at (167.2, 108.7)
- added D2: SS34, Diode_SMD:D_SMA, F.Cu at (167.8, 105.8)
- added D4: SS34, Diode_SMD:D_SMA, F.Cu at (171.3, 95.3)
- added J12: Barrel_Jack_MountingPin, Connector_BarrelJack:BarrelJack_Wuerth_6941xx301002, F.Cu at (165.6, 118.0)
- added L1: 10uH, Inductor_SMD:L_Coilcraft_XxL4020, F.Cu at (163.8, 101.5)
- added R5: 10k, Resistor_SMD:R_0603_1608Metric, F.Cu at (173.8, 102.6)
- added R6: 31.6k, Resistor_SMD:R_0603_1608Metric, F.Cu at (172.4, 105.2)
- added R7: 1M, Resistor_SMD:R_0603_1608Metric, F.Cu at (173.6, 99.2)
- C2: value 100n -> 10u; footprint Capacitor_SMD:C_0603_1608Metric -> Capacitor_SMD:C_0805_2012Metric
- C3: value 1uF -> 100n; footprint Capacitor_Tantalum_SMD:CP_EIA-3528-21_Kemet-B -> Capacitor_SMD:C_0603_1608Metric
- R1, R4, R8, R9: value 11k -> 10k
- U2: value LM317AG-TN3-R -> ME3116; footprint Package_TO_SOT_SMD:TO-252-2 -> Package_TO_SOT_SMD:SOT-23-6
- moved D3 46.8 mm to (164.8, 78.5)
- moved R3 46.8 mm to (164.8, 81.8)
- moved SW1 42.8 mm to (113.5, 94.3)
- moved D1 39.5 mm to (160.2, 78.4)
- moved R2 39.5 mm to (160.2, 81.8)
- moved R9 11.3 mm to (118.5, 92.0), turned to 90 degrees
- moved C2 10.2 mm to (167.3, 98.1), turned to 0 degrees
- moved Ref** 8.75 mm to (112.2, 111.5)
- moved C3 6.86 mm to (170.9, 98.1), turned to 0 degrees
- moved J10 5.00 mm to (160.2, 124.2)
- moved J6 5.00 mm to (120.2, 124.2)
- moved J7 5.00 mm to (130.2, 124.2)
- moved J8 5.00 mm to (140.2, 124.2)
- moved J9 5.00 mm to (150.2, 124.2)
- moved U2 1.42 mm to (170.2, 101.2)
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Connections:
- C10 pad 1: 3v3VD -> +3V3
- C11 pad 1: 3v3VD -> +3V3
- C12 pad 1: 3v3VD -> +3V3
- C2 pad 1: 5V -> GND
- C2 pad 2: GND -> Net-(C2-Pad2)
- C3 pad 1: 3v3VD -> Net-(C2-Pad2)
- D3 pad 2: 3v3VD -> +3V3
- J1 pad 3: 3v3VD -> +3V3
- J10 pad 3: 3v3VD -> +3V3
- J2 pad 3: 3v3VD -> +3V3
- J3 pad 3: 3v3VD -> +3V3
- J4 pad 3: 3v3VD -> +3V3
- J5 pad 3: 3v3VD -> +3V3
- J6 pad 3: 3v3VD -> +3V3
- J7 pad 3: 3v3VD -> +3V3
- J8 pad 3: 3v3VD -> +3V3
- J9 pad 3: 3v3VD -> +3V3
- R1 pad 1: 3v3VD -> +3V3
- R8 pad 1: 3v3VD -> +3V3
- R9 pad 2: 3v3VD -> +3V3
- U1 pad 2: 3v3VD -> +3V3
- U2 pad 2: 3v3VD -> GND
- U2 pad 3: 5V -> Net-(C4-Pad1)
- U5 pad 5: 3v3VD -> +3V3
Routing:
- net 3v3VD: track 266.3 -> 0.00 mm
- net +3V3: track 0.00 -> 254.6 mm
- net Net-(C2-Pad2): track 0.00 -> 39.7 mm, vias 0 -> 2
- net P10: track 84.6 -> 64.0 mm
- net SYS_OK_LED: track 37.6 -> 23.1 mm
- net 5V: track 18.6 -> 7.15 mm
- net Net-(C5-Pad1): track 0.00 -> 9.51 mm
- net GND: track 38.9 -> 48.3 mm, vias 55 -> 114
- net RST: track 35.9 -> 26.5 mm
- net Net-(C4-Pad1): track 0.00 -> 6.31 mm
- net P9: track 46.8 -> 51.0 mm
- net Net-(C5-Pad2): track 4.44 -> 1.93 mm
- net P7: track 56.2 -> 58.6 mm
- net Net-(R7-Pad2): track 0.00 -> 2.41 mm
- net D-: track 5.22 -> 7.42 mm
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Other:
- board text added: "ESP32_Smart_Keezer: Rev 1 Acea Quigg 8/21"
- board text removed: "ESP32_Smart_Keezer: Rev 0"

Commit message: Rev 1 - WIP
Parts:
- moved C6 14.2 mm to (171.0, 95.0)
- moved C5 12.1 mm to (167.8, 113.3), turned to 0 degrees
- moved R5 10.1 mm to (174.2, 112.7), turned to 90 degrees
- moved L1 8.66 mm to (167.0, 109.5)
- moved C4 8.50 mm to (170.7, 113.0)
- moved D2 8.10 mm to (171.2, 98.5)
- moved U2 7.85 mm to (172.4, 108.8)
- moved R6 7.50 mm to (172.6, 112.7)
- moved C3 7.28 mm to (171.6, 105.3)
- moved C2 6.33 mm to (171.3, 103.0), turned to 180 degrees
- moved D4 5.73 mm to (165.7, 94.7), turned to 90 degrees
- moved R7 3.72 mm to (170.4, 101.2), turned to 0 degrees
- moved J12 3.36 mm to (165.4, 121.3)
Routing:
- net Net-(C5-Pad1): track 9.51 -> 0.00 mm
- net GND: track 48.3 -> 40.5 mm, vias 114 -> 121
- net +3V3: track 254.6 -> 261.8 mm, vias 0 -> 4
- net Net-(R7-Pad2): track 2.41 -> 7.29 mm
- net Net-(C2-Pad2): track 39.7 -> 36.1 mm, vias 2 -> 3
- net Net-(C5-Pad2): track 1.93 -> 5.12 mm
- net P8: track 67.4 -> 66.0 mm
- net P9: track 51.0 -> 50.4 mm
- added copper zone on F.Cu, net Net-(C2-Pad2)
- added copper zone on F.Cu, net Net-(C5-Pad1)
Other:
- net class Default: clearance 0.2 -> 0.167; via_dia 0.8 -> 0.6
- rule trace_clearance: 0.2 -> 0.167

Commit message: REV 1 - off to JLCPCB
Parts:
- removed C4: 0.47uF, Capacitor_SMD:C_0805_2012Metric
- removed C5: 10u, Capacitor_SMD:C_0805_2012Metric
- removed R5: 10k, Resistor_SMD:R_0603_1608Metric
- removed R6: 31.6k, Resistor_SMD:R_0603_1608Metric
- C2: value 10u -> 220uF; footprint Capacitor_SMD:C_0805_2012Metric -> Capacitor_SMD:C_Elec_6.3x7.7
- C6: value 10u -> 220uF; footprint Capacitor_SMD:C_0805_2012Metric -> Capacitor_Tantalum_SMD:CP_EIA-3528-15_AVX-H
- L1: value 10uH -> 47uH; footprint Inductor_SMD:L_Coilcraft_XxL4020 -> Inductor_SMD:L_Bourns_SRN6045TA
- U2: value ME3116 -> XL1509_SOP8; footprint Package_TO_SOT_SMD:SOT-23-6 -> Package_SO:SOIC-8_3.9x4.9mm_P1.27mm
- U5: value CH330N -> CH340N
- moved R7 10.0 mm to (169.8, 111.2), turned to 180 degrees
- moved C6 9.51 mm to (161.7, 96.8), turned to 90 degrees
- moved L1 9.18 mm to (160.1, 103.5), turned to 90 degrees
- moved D2 6.67 mm to (165.7, 102.2), turned to 90 degrees
- moved C2 5.46 mm to (171.7, 97.5), turned to 270 degrees
- moved C3 2.21 mm to (170.7, 103.3)
- moved U2 1.81 mm to (171.2, 107.3), turned to 0 degrees
- moved D4 0.20 mm to (165.8, 94.7)
Connections:
- C2 pad 1: GND -> VIN
- C2 pad 2: Net-(C2-Pad2) -> GND
- C3 pad 1: Net-(C2-Pad2) -> VIN
- D2 pad 1: Net-(C5-Pad1) -> +3V3
- D4 pad 1: Net-(C2-Pad2) -> VIN
- J12 pad 1: Net-(C2-Pad2) -> VIN
- L1 pad 1: Net-(C5-Pad1) -> Net-(L1-Pad1)
- R7 pad 1: Net-(C2-Pad2) -> VIN
- U2 pad 1: Net-(C5-Pad2) -> VIN
- U2 pad 2: GND -> +3V3
- U2 pad 3: Net-(C4-Pad1) -> Net-(L1-Pad1)
- U2 pad 5: Net-(C2-Pad2) -> GND
- U2 pad 6: Net-(C5-Pad1) -> GND
- U5 pad 4: (no net) -> RST
Routing:
- net Net-(C2-Pad2): track 36.1 -> 0.00 mm, vias 3 -> 0
- net RST: track 26.5 -> 61.5 mm, vias 0 -> 2
- net VIN: track 0.00 -> 33.4 mm
- net +3V3: track 261.8 -> 249.1 mm, vias 4 -> 8
- net Net-(L1-Pad1): track 0.00 -> 8.73 mm
- net Net-(C4-Pad1): track 6.59 -> 0.00 mm
- net Net-(R7-Pad2): track 7.29 -> 2.00 mm
- net Net-(C5-Pad2): track 5.12 -> 0.00 mm
- net GND: track 40.5 -> 36.2 mm, vias 121 -> 126
- added copper zone on F.Cu, net +3V3
- added copper zone on F.Cu, net Net-(L1-Pad1)
- removed copper zone on F.Cu, net Net-(C2-Pad2)
- removed copper zone on F.Cu, net Net-(C5-Pad1)

Commit message: Cleaning up
Parts:
- moved D2 8.05 mm to (157.7, 103.0), turned to 270 degrees
- moved L1 3.51 mm to (163.6, 103.3)
Connections:
- U2 pad 2: +3V3 -> Net-(L1-Pad1)
- U2 pad 3: Net-(L1-Pad1) -> +3V3
Routing:
- net +3V3: track 249.1 -> 270.2 mm, vias 8 -> 10
- net Net-(L1-Pad1): track 8.73 -> 1.16 mm
- net GND: track 36.2 -> 33.8 mm, vias 126 -> 127
- net P8: track 66.0 -> 67.0 mm
- removed copper zone on F.Cu, net +3V3
