File: PCBs/keezer_pcb/esp32_smart_keezer.sch (KiCad schematic (older format))
At the start: 34 parts, among them J1 Conn_01x03_Male, J10 Conn_01x03_Male, J11 USB_B_Micro, J2 Conn_01x03_Male, J3 Conn_01x03_Male, J4 Conn_01x03_Male, J5 Conn_01x03_Male, J6 Conn_01x03_Male, J7 Conn_01x03_Male, J8 Conn_01x03_Male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

Commit message: Rev 1 - WIP
Parts:
- removed C3: 1uF, Capacitor_Tantalum_SMD:CP_EIA-3528-21_Kemet-B, symbol Device:CP_Small
- removed R25: 200R, Resistor_SMD:R_0603_1608Metric, symbol Device:R_Small
- removed R26: 330R, Resistor_SMD:R_0603_1608Metric, symbol Device:R_Small
- removed U2: LM317AG-TN3-R, Package_TO_SOT_SMD:TO-252-2, symbol Regulator_Linear:LM317_TO-252
- added C3: 100n, Capacitor_SMD:C_0603_1608Metric, symbol Device:C_Small
- added C4: 0.47uF, Capacitor_SMD:C_0805_2012Metric, symbol Device:C_Small
- added C5, C6: 10u, Capacitor_SMD:C_0805_2012Metric, symbol Device:C_Small
- added D2, D4: SS34, Diode_SMD:D_SMA, symbol Diode:1N4148WS
- added J12: Barrel_Jack_MountingPin, Connector_BarrelJack:BarrelJack_Wuerth_6941xx301002, symbol Connector:Barrel_Jack_MountingPin
- added L1: 10uH, Inductor_SMD:L_Coilcraft_XxL4020, symbol Device:L_Small
- added R5: 10k, Resistor_SMD:R_0603_1608Metric, symbol Device:R_Small
- added R6: 31.6k, Resistor_SMD:R_0603_1608Metric, symbol Device:R_Small
- added R7: 1M, Resistor_SMD:R_0603_1608Metric, symbol Device:R_Small
- added U2: ME3116, Package_TO_SOT_SMD:SOT-23-6, symbol me3116:ME3116
- C2: value 100n -> 10u; footprint Capacitor_SMD:C_0603_1608Metric -> Capacitor_SMD:C_0805_2012Metric; lcsc_part_number C14663 -> C15850; lcsc_url https://lcsc.com/product-detail/Multilayer-Ceramic-Capacito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 -> (none); package 0603 -> (none)
- R1, R4, R8, R9: value 11k -> 10k; lcsc_part_number C25950 -> C25804; lcsc_url https://lcsc.com/product-detail/Chip-Resistor-Surface-Mount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 -> (none)
Connections:
- net +3V3: now also C4.2, C6.1, L1.2, R6.1
- net 5V: now also D4.2 (A); no longer C2.1
- net GND: now also C2.1, C3.2, C6.2, D2.2 (A), J12.2, R5.2, U2.2 (GND); no longer C2.2
- new net: C2.2, C3.1, D4.1 (K), J12.1, R7.1, U2.5 (IN)
- new net: C5.1, D2.1 (K), L1.1, U2.6 (SW)
- new net: C4.1, R5.1, R6.2, U2.3 (FB)
- new net: C5.2, U2.1 (BS)
- new net: R7.2, U2.4 (EN)
- no-connect marks 19 -> 20
Other:
- note added: "DC-DC Buck (40V to 3.3V 600mA)"
- note removed: "DC-DC Buck (30V, 3.3V, 1.5A)"
- moved on the sheet: D1, D3, J11, R2, R3

Commit message: Rev 1 - WIP
Parts:
- C4: footprint Capacitor_SMD:C_0805_2012Metric -> Capacitor_SMD:C_0201_0603Metric
Changed lines of the file:
@@
 F 0 "C4" H 3700 1750 50  0000 L CNN
 F 1 "0.47uF" H 3550 1900 50  0000 L CNN
-F 2 "Capacitor_SMD:C_0805_2012Metric" H 3850 1800 50  0001 C CNN
+F 2 "Capacitor_SMD:C_0201_0603Metric" H 3850 1800 50  0001 C CNN
 F 3 "" H 3850 1800 50  0001 C CNN
 F 4 "C1623" H 3850 1800 50  0001 C CNN "lcsc_part_number"

Commit message: REV 1 - off to JLCPCB
Parts:
- removed C2, C5, C6: 10u, Capacitor_SMD:C_0805_2012Metric, symbol Device:C_Small
- removed C4: 0.47uF, Capacitor_SMD:C_0201_0603Metric, symbol Device:C_Small
- removed D2: SS34, Diode_SMD:D_SMA, symbol Diode:1N4148WS
- removed R5: 10k, Resistor_SMD:R_0603_1608Metric, symbol Device:R_Small
- removed R6: 31.6k, Resistor_SMD:R_0603_1608Metric, symbol Device:R_Small
- removed U2: ME3116, Package_TO_SOT_SMD:SOT-23-6, symbol me3116:ME3116
- added C2: 220uF, Capacitor_SMD:C_Elec_6.3x7.7, symbol Device:CP_Small
- added C6: 220uF, Capacitor_Tantalum_SMD:CP_EIA-3528-15_AVX-H, symbol Device:CP_Small
- added D2: SS34, Diode_SMD:D_SMA, symbol Device:D_Small
- added U2: XL1509_SOP8, Package_SO:SOIC-8_3.9x4.9mm_P1.27mm, symbol xl1509_sop8:XL1509_SOP8
- L1: value 10uH -> 47uH; footprint Inductor_SMD:L_Coilcraft_XxL4020 -> Inductor_SMD:L_Bourns_SRN6045TA; lcsc_part_number C408339 -> C36414
- U5: value CH330N -> CH340N; lcsc_part_number C108996 -> C506813; lcsc_url https://lcsc.com/product-detail/USB-ICs_WCH-Jiangsu-Qin-Hen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 -> (none); mfr_part_number CH330N -> CH340N
Connections:
- net labels added: +3.3V, VIN
- wire segments 50 -> 49
- no-connect marks 20 -> 19
Other:
- moved on the sheet: C3, D4, J12, R7

Commit message: Cleaning up
Other:
- moved on the sheet: L1
Changed lines of the file:
@@
 Sheet 1 1
 Title "ESP32 Smart Keezer"
-Date "2021-08-28"
-Rev "1"
+Date "2021-09-22"
+Rev "2"
 Comp "Acea Quigg"
 Comment1 ""
@@
 L Device:L_Small L1
 U 1 1 6132B509
-P 2575 1669
-F 0 "L1" V 2775 1669 50  0000 C CNN
-F 1 "47uH" V 2675 1669 50  0000 C CNN
-F 2 "Inductor_SMD:L_Bourns_SRN6045TA" H 2575 1669 50  0001 C CNN
-F 3 "~" H 2575 1669 50  0001 C CNN
-F 4 "C36414" H 2575 1669 50  0001 C CNN "lcsc_part_number"
-	1    2575 1669
+P 2544 1769
+F 0 "L1" V 2488 1765 50  0000 C CNN
+F 1 "47uH" V 2398 1772 50  0000 C CNN
+F 2 "Inductor_SMD:L_Bourns_SRN6045TA" H 2544 1769 50  0001 C CNN
+F 3 "~" H 2544 1769 50  0001 C CNN
+F 4 "C36414" H 2544 1769 50  0001 C CNN "lcsc_part_number"
+	1    2544 1769
 	0    -1   -1   0
 $EndComp
-Wire Wire Line
-	2675 1669 2975 1669
 Wire Wire Line
 	2975 1669 2975 1769
@@
 Connection ~ 3175 1769
 Wire Wire Line
-	2325 1769 2975 1769
-Wire Wire Line
-	2475 1669 2325 1669
-Wire Wire Line
 	2325 1569 2402 1569
 Wire Wire Line
@@
 Text GLabel 10438 1680 2    50   Input ~ 0
 RST
+Wire Wire Line
+	2325 1769 2444 1769
+Wire Wire Line
+	2644 1769 2975 1769
+Wire Wire Line
+	2325 1669 2975 1669
 $EndSCHEMATC
